File: Schematics/new/drv8711/drv8711.sch (KiCad schematic (older format))
At the start: 11 parts

Commit message: add new project, edit schematics
Parts:
- added C? (x6): C, symbol Device:C
- added C?: CP, symbol Device:CP
- added R? (x4): R_Small, symbol Device:R_Small
- added RN? (x2): R_Pack04, symbol Device:R_Pack04
Connections:
- net VDD: now reaches U?.1 (VDD)
- net VDD: now also U?.17 (VDD), U?.5 (VDDA), R?.2, RN?.2 (R2.1), RN?.3 (R3.1)
- net at U?.10 (PA4): now also RN?.3 (R3.1)
- net at U?.11 (PA5): now also RN?.1 (R1.1)
- net at U?.12 (PA6): now also RN?.4 (R4.1)
- net at U?.13 (PA7): now also RN?.2 (R2.1)
- net GNDD: now reaches U?.16 (VSS)
- net GNDD: now also U?.32 (VSS)
- net at U?.19 (PA9): now also RN?.4 (R4.1)
- net at U?.20 (PA10): now also RN?.1 (R1.1)
- net at U?.1 (CP1): now also C?.1
- net at U?.14 (SCLK): now also RN?.8 (R1.2)
- net at U?.15 (SDATI): now also RN?.7 (R2.2)
- net at U?.16 (SCS): now also RN?.6 (R3.2)
- net at U?.17 (SDATO): now also RN?.5 (R4.2)
- net at U?.18 (FAULTn): now also RN?.7 (R2.2), RN?.8 (R1.2)
- net at U?.19 (STALLn/BEMFVn): now also RN?.5 (R4.2), RN?.6 (R3.2)
- net at U?.2 (CP2): now also C?.2
- net at U?.20 (BEMF): now also C?.1
- net at U?.21 (BOUT2): now also Q?.2 (D), Q?.3 (S)
- net at U?.22 (B2HS): now also Q?.1 (G)
- net at U?.23 (B2LS): now also Q?.1 (G)
- net GND: now reaches U?.24 (BISENN)
- net GND: now also U?.29 (GND), U?.33 (AISENN), U?.38 (GND), U?.39 (GND), U?.5 (GND), C?.1, C?.2, C?.2, C?.2, C?.2, R?.1, R?.1, R?.2
- net at U?.25 (BISENP): now also Q?.3 (S), Q?.3 (S), R?.2
- net at U?.26 (B1LS): now also Q?.1 (G)
- net at U?.27 (B1HS): now also Q?.1 (G)
- net at U?.28 (BOUT1): now also Q?.2 (D), Q?.3 (S)
- net at U?.3 (VCP): now also C?.1
- net at U?.30 (AOUT2): now also Q?.2 (D), Q?.3 (S)
- net at U?.31 (A2HS): now also Q?.1 (G)
- net at U?.32 (A2LS): now also Q?.1 (G)
- net at U?.34 (AISENP): now also Q?.3 (S), Q?.3 (S), R?.2
- net at U?.35 (A1LS): now also Q?.1 (G)
- net at U?.36 (A1HS): now also Q?.1 (G)
- net at U?.37 (AOUT1): now also Q?.2 (D), Q?.3 (S)
- net +VDC: now reaches U?.4 (VM)
- net +VDC: now also Q?.2 (D), Q?.2 (D), Q?.2 (D), Q?.2 (D), C?.1, C?.1, C?.2
- net at U?.6 (V5): now also C?.1
- net at U?.7 (VINT): now also C?.2
- net at U?.8 (SLEEPn): now also R?.1
- net at U?.9 (RESET): now also R?.1
Other:
- moved on the sheet: Q?, U?
